Commit message: 增加gazebo仿真场景 便于提前验证算法

File: src/dashgo_description/urdf/dashgobase/base.urdf.xacro (robot description, xacro)
@@ -6,7 +6,9 @@
   <xacro:property name="base_length" value="0.20" />
   <xacro:property name="wheel_length" value="0.046" />
-  <xacro:property name="wheel_radius" value="0.062" />
+  <!-- Keep the displayed/physical wheel geometry aligned with the calibrated
+       values used by dashgo_driver/config/base.yaml. -->
+  <xacro:property name="wheel_radius" value="0.074" />
   <xacro:property name="wheel_offset_x" value="-0.08" />
-  <xacro:property name="wheel_offset_y" value="0.176" />
+  <xacro:property name="wheel_offset_y" value="0.2225" />
   <xacro:property name="wheel_offset_z" value="-0.038" />
   <xacro:property name="PI" value="3.1415926" />
@@ -16,6 +18,10 @@
       <axis xyz="0 0 1" />
       <limit effort="100" velocity="100"/>
+      <dynamics damping="0.2" friction="0.05" />
       <safety_controller k_velocity="10" />
-      <origin xyz="${wheel_offset_x} ${reflect*wheel_offset_y} ${wheel_offset_z}" rpy="${reflect*PI/2} 0 0" />
+      <!-- Both wheel joint axes must point in the same base-frame direction;
+           mirroring the cylinder rotation would make equal Gazebo wheel
+           velocities rotate the chassis instead of driving it straight. -->
+      <origin xyz="${wheel_offset_x} ${reflect*wheel_offset_y} ${wheel_offset_z}" rpy="${-PI/2} 0 0" />
       <parent link="${parent}_link"/>
       <child link="${parent}_${suffix}_wheel_link"/>
@@ -39,4 +45,18 @@
         <material name="${color}" />
       </visual>
+      <collision>
+        <origin xyz="0 0 0" rpy="0 0 0" />
+        <geometry>
+          <cylinder radius="${wheel_radius}" length="${wheel_length}"/>
+        </geometry>
+      </collision>
+      <!-- Idealized wheel mass/inertia for Gazebo. The measured drivetrain
+           dimensions above remain the parameters relevant to kinematics. -->
+      <inertial>
+        <origin xyz="0 0 0" rpy="0 0 0" />
+        <mass value="0.5" />
+        <inertia ixx="0.001011" ixy="0" ixz="0"
+                 iyy="0.001011" iyz="0" izz="0.001369" />
+      </inertial>
     </link>
   </xacro:macro>
@@ -62,5 +82,5 @@
                 <box size="${base_x} ${base_y} ${base_length}"/>
             </geometry>
-            <material name="iRobot/LightGrey"/>
+            <material name="Grey"/>
         </visual>
         <collision>
@@ -70,4 +90,12 @@
             </geometry>
         </collision>
+        <!-- Idealized chassis mass/inertia. Replace these values when measured
+             data is available; dimensions intentionally retain the old box. -->
+        <inertial>
+            <origin xyz="0 0 0" rpy="0 0 0"/>
+            <mass value="20.0"/>
+            <inertia ixx="0.333333" ixy="0" ixz="0"
+                     iyy="0.333333" iyz="0" izz="0.533333"/>
+        </inertial>
     </link>
   </xacro:macro>

Commit message: 修复仿真中雷达自体回波

File: src/dashgo_description/urdf/dashgobase/base.urdf.xacro (robot description, xacro)
@@ -2,7 +2,10 @@
 <robot name="base" xmlns:xacro="http://ros.org/wiki/xacro">
   <!-- Define a number of dimensions using properties -->
-  <xacro:property name="base_x" value="0.40" />
-  <xacro:property name="base_y" value="0.40" />
+  <!-- Measured outer chassis/wheel envelope, shared with the navigation
+       footprint: [-0.283, 0.283] in base_footprint. -->
+  <xacro:property name="base_x" value="0.566" />
+  <xacro:property name="base_y" value="0.566" />
   <xacro:property name="base_length" value="0.20" />
+  <xacro:property name="base_link_offset_x" value="0.115" />
   <xacro:property name="wheel_length" value="0.046" />
   <!-- Keep the displayed/physical wheel geometry aligned with the calibrated
@@ -78,5 +81,6 @@
 -->
         <visual>
-            <origin xyz="0 0 0" rpy="0 0 0"/>
+            <!-- base_link is 0.115 m ahead of the measured footprint center. -->
+            <origin xyz="${-base_link_offset_x} 0 0" rpy="0 0 0"/>
             <geometry>
                 <box size="${base_x} ${base_y} ${base_length}"/>
@@ -85,16 +89,16 @@
         </visual>
         <collision>
-            <origin xyz="0 0 0" rpy="0 0 0"/>
+            <origin xyz="${-base_link_offset_x} 0 0" rpy="0 0 0"/>
             <geometry>
                  <box size="${base_x} ${base_y} ${base_length}"/>
             </geometry>
         </collision>
-        <!-- Idealized chassis mass/inertia. Replace these values when measured
-             data is available; dimensions intentionally retain the old box. -->
+        <!-- Idealized uniform-box chassis mass/inertia. Its center is aligned
+             with the measured footprint center; replace when measured. -->
         <inertial>
-            <origin xyz="0 0 0" rpy="0 0 0"/>
+            <origin xyz="${-base_link_offset_x} 0 0" rpy="0 0 0"/>
             <mass value="20.0"/>
-            <inertia ixx="0.333333" ixy="0" ixz="0"
-                     iyy="0.333333" iyz="0" izz="0.533333"/>
+            <inertia ixx="0.600593" ixy="0" ixz="0"
+                     iyy="0.600593" iyz="0" izz="1.067853"/>
         </inertial>
     </link>
@@ -113,5 +117,6 @@
     <origin xyz="0 0 0.04" rpy="0 0 0" />
 -->
-    <origin xyz="0.115 0 ${base_length/2 - wheel_offset_z}" rpy="0 0 0" />
+    <!-- Put base_footprint on the drive-wheel contact plane. -->
+    <origin xyz="${base_link_offset_x} 0 ${wheel_radius - wheel_offset_z}" rpy="0 0 0" />
     <parent link="base_footprint"/>
     <child link="base_link" />

File: src/dashgo_description/urdf/dashgobase/dashgobase.xacro (robot description, xacro)
@@ -49,5 +49,6 @@
   </link>
   <joint name="front_point_flag" type="fixed">
-    <origin xyz="0.2 0 ${base_length/2}" rpy="0 0 0" />
+    <!-- Keep the marker on the measured +0.283 m footprint boundary. -->
+    <origin xyz="${base_x/2 - base_link_offset_x} 0 ${base_length/2}" rpy="0 0 0" />
     <parent link="base_link"/>
     <child link="front_flag" />

File: src/dashgo_gazebo/urdf/dashgo.gazebo.xacro (robot description, xacro)
@@ -1,5 +1,5 @@
 <?xml version="1.0"?>
 <robot name="dashgo_sim" xmlns:xacro="http://ros.org/wiki/xacro">
-  <!-- The shared description contains the 0.40 x 0.40 m chassis, two drive
+  <!-- The shared description contains the measured 0.566 x 0.566 m envelope, two drive
        wheels, base frames and RViz visuals. -->
   <xacro:include filename="$(find dashgo_description)/urdf/dashgobase/dashgobase.xacro" />
@@ -42,8 +42,18 @@
     </gazebo>
   </xacro:macro>
-  <xacro:omni_support name="front_left_omni" x="0.17" y="0.17" />
-  <xacro:omni_support name="front_right_omni" x="0.17" y="-0.17" />
-  <xacro:omni_support name="rear_left_omni" x="-0.17" y="0.17" />
-  <xacro:omni_support name="rear_right_omni" x="-0.17" y="-0.17" />
+  <!-- Sphere centers are one radius inside the measured +/-0.283 m envelope.
+       X values are converted from base_footprint to the offset base_link. -->
+  <xacro:omni_support name="front_left_omni"
+                      x="${base_x/2 - support_radius - base_link_offset_x}"
+                      y="${base_y/2 - support_radius}" />
+  <xacro:omni_support name="front_right_omni"
+                      x="${base_x/2 - support_radius - base_link_offset_x}"
+                      y="${-base_y/2 + support_radius}" />
+  <xacro:omni_support name="rear_left_omni"
+                      x="${-base_x/2 + support_radius - base_link_offset_x}"
+                      y="${base_y/2 - support_radius}" />
+  <xacro:omni_support name="rear_right_omni"
+                      x="${-base_x/2 + support_radius - base_link_offset_x}"
+                      y="${-base_y/2 + support_radius}" />
   <gazebo reference="base_link">
     <material>Gazebo/Grey</material>
@@ -129,12 +139,15 @@
        obstacle band, but is high enough that a small chassis pitch cannot make
        the horizontal rays intersect the ground plane. -->
-  <xacro:sim_laser name="laser_frame" topic="scan"
-                   xyz="0.059 -0.176 0.142" rpy="0 0 -0.785"
+  <!-- Keep Gazebo's unfiltered main scan separate. sim_robot.launch removes
+       returns inside the retained chassis envelope and republishes /scan for
+       mapping, navigation and the safety gate. -->
+  <xacro:sim_laser name="laser_frame" topic="scan_raw"
+                   xyz="0.059 -0.176 0.168" rpy="0 0 -0.785"
                    min_angle="-2.356194" max_angle="2.356194" samples="1080" />
   <xacro:sim_laser name="laser_frame_2" topic="scan_2"
-                   xyz="0.250 0 -0.070" rpy="0 3.141592654 -3.04"
+                   xyz="0.250 0 -0.044" rpy="0 3.141592654 -3.04"
                    min_angle="-1.570796" max_angle="1.570796" samples="720" />
   <xacro:sim_laser name="laser_frame_3" topic="scan_3"
-                   xyz="-0.289 0.176 0.212" rpy="0 0 2.355"
+                   xyz="-0.289 0.176 0.238" rpy="0 0 2.355"
                    min_angle="-2.356194" max_angle="2.094395" samples="1020" />
   <gazebo reference="base_link">
